Commit message: create mobility lab local version for the pull-over function

File: example_calibration_folder/vehicle/calibration/urdf/carma.urdf (robot description, URDF)
Before this commit: robot vehicle_platform, 13 links, 12 joints
Links:
- removed link novatel_gnss
- added link gps
Joints:
- removed joint lidar
- added joint velodyne: type fixed, parent base_link, child velodyne, origin xyz=1.02 0 2.23 rpy=0 0 0
- joint base_link_to_novatel: child novatel_gnss -> gps
- joint gnss_to_ned_heading: parent novatel_gnss -> gps
